File: Circuit/connection board/Connection Board.sch (KiCad schematic (older format))
At the start: 6 parts, among them J1 BME280, J2 BH1750, J3 Sensirion SPS30, J4 OLED 1.3\" i2c, U1 WeMos_D1_mini

Commit message: Added case and yaml code
Other:
- note added: "Luminance"
- note removed: "Illuminance"
Changed lines of the file:
@@
 Temp/Press/Humi
 Text Notes 5475 825  0    118  ~ 24
-Illuminance
+Luminance
 Text Notes 7625 825  0    118  ~ 24
 Air Quality
